Commit message: tiago kinematics only fixed

File: config/fake_ros2_control.urdf.xacro (robot description, xacro)
@@ -14,5 +14,5 @@
 <robot xmlns:xacro="http://ros.org/wiki/xacro"
        name="tiago" >
-  <xacro:macro name="tiago_ros2_control" params="use_sim:=^|true">
+  <xacro:macro name="tiago_ros2_control" params="use_sim:=^|false">
     <xacro:arg name="arm" default="true" />
     <xacro:arg name="end_effector" default="pal-hey5"/>
@@ -30,5 +30,8 @@
       </xacro:if>
       <xacro:if value="${end_effector == 'pal-hey5'}">
-        <xacro:include filename="$(find hey5_description)/urdf/hey5.ros2_control.xacro" />
+        <xacro:include filename="$(find pal_hey5_description)/urdf/pal_hey5.ros2_control.xacro" />
+      </xacro:if>
+      <xacro:if value="${end_effector in ['robotiq-2f-85', 'robotiq-2f-140']}">
+        <xacro:include filename="$(find pal_robotiq_description)/urdf/robotiq.ros2_control.xacro" />
       </xacro:if>
     </xacro:if>
@@ -78,11 +81,17 @@
           <xacro:ros2_control_hey5 name="hand"/>
         </xacro:if>
+        <xacro:if value="${end_effector == 'robotiq-2f-85'}">
+          <!-- robotiq-2f-85 -->
+          <xacro:ros2_control_robotiq_85_gripper name="gripper" reduction="1.0" />
+        </xacro:if>
+        <xacro:if value="${end_effector == 'robotiq-2f-140'}">
+          <!-- robotiq-2f-140 -->
+          <xacro:ros2_control_robotiq_140_gripper name="gripper" reduction="1.0" />
+        </xacro:if>
       </xacro:if>
       <!-- Force Torque sensor -->
       <xacro:if value="${has_ft_sensor}">
         <xacro:include filename="$(find tiago_description)/urdf/sensors/sensors.ros2_control.xacro"/>
-        <xacro:if value="$(arg use_sim)">
-          <xacro:ros2_control_force_torque_sensor name="wrist_ft_joint_force_torque"/>
-        </xacro:if>
+        <xacro:ros2_control_force_torque_sensor name="wrist_ft_sensor"/>
       </xacro:if>
     </ros2_control>

File: config/tiago_fake.urdf.xacro (robot description, xacro)
@@ -14,7 +14,7 @@
 <robot  xmlns:xacro="http://ros.org/wiki/xacro"
         name="tiago" >
-    <xacro:arg name="arm" default="right-arm"/> <!-- right-arm, no-arm -->
+    <xacro:arg name="arm" default="tiago-arm"/> <!-- tiago-arm, no-arm -->
     <xacro:arg name="wrist_model" default="wrist-2010"/>
-    <xacro:arg name="end_effector" default="pal-gripper"/> <!-- no-end-effector, pal-gripper, pal-hey5-->
+    <xacro:arg name="end_effector" default="pal-hey5"/> <!-- no-end-effector, pal-gripper, pal-hey5-->
     <xacro:arg name="ft_sensor" default="schunk-ft"/> <!-- no-ft-sensor, schunk-ft -->
     <xacro:arg name="laser_model" default="sick-571"/> <!-- no-laser, hokuyo, sick-551, sick-561, sick-571-->
@@ -28,5 +28,5 @@
     <xacro:arg name="use_sim" default="false"/>
     <xacro:property name="arm" value="$(arg arm)" />
-    <xacro:if value="${arm not in ['right-arm', 'no-arm']}">
+    <xacro:if value="${arm not in ['right-arm', 'tiago-arm', 'no-arm']}">
       <xacro:wrong_arm/>
     </xacro:if>
@@ -45,5 +45,5 @@
     </xacro:if>
   </xacro:if>
-  <xacro:if value="${end_effector not in ['no-end-effector', 'pal-gripper', 'pal-hey5', 'custom']}">
+  <xacro:if value="${end_effector not in ['no-end-effector', 'pal-gripper', 'pal-hey5', 'custom', 'robotiq-2f-85', 'robotiq-2f-140']}">
     <xacro:wrong_end_effector/>
   </xacro:if>
@@ -90,5 +90,5 @@
     use_sim="$(arg use_sim)" />
   <!-- Materials for visualization -->
-  <xacro:include filename="$(find tiago_description)/urdf/materials.urdf.xacro" />
+  <xacro:include filename="$(find pal_urdf_utils)/urdf/materials.urdf.xacro" />
   <!-- Now we can start using the macros included above to define the actual robot -->
   <xacro:base_sensors name="base" laser_model="$(arg laser_model)" sonars="true" microphone="true"/>
@@ -107,4 +107,5 @@
   <xacro:if value="${has_ft_sensor}">
       <xacro:ft_sensor name="wrist" parent="arm_tool_link" />
+      <xacro:force_torque_sensor_gazebo name="wrist_ft" update_rate="100"/>
   </xacro:if>
   <!-- Thermal camera -->
