Commit message: steam deck added

File: config/tiago_fake.urdf.xacro (robot description, xacro)
@@ -137,3 +137,22 @@
       </inertial>
   </link>
+  <!-- Steam deck -->
+  <joint name="steamdeck_joint" type="fixed">
+      <parent link="torso_lift_link"/>
+      <child link="steamdeck_link"/>
+      <origin xyz="0.275 0 -0.0585" rpy="0 -0.122173 0" />
+  </joint>
+  <link name="steamdeck_link">
+    <inertial>
+      <origin xyz="0 0 0" rpy="0 0 0"/>
+      <mass value="0.0001" />
+      <inertia ixx="0.0001"  ixy="0"  ixz="0" iyy="0.0001" iyz="0" izz="0.0001" />
+    </inertial>
+    <collision>
+      <origin xyz="0 0 0" rpy="0 0 0"/>
+      <geometry>
+        <box size="0.05 0.298 0.117"/>
+      </geometry>
+    </collision>
+  </link>
 </robot>
